File: Tarea 5/PLC4UNI-GC1_PCB-main/PLC4UNI-GC1_PCB-main/PLC4UNI-GC1_PCB/PLC4UNI-GC1.kicad_pcb (KiCad board)
At the start: 4 copper layers, 102.4 x 83.1 mm, 205 parts, among them J1 Conn_02x08_Odd_Even, J2 Screw_Terminal_9_P5.00mm, J3 Screw_Terminal_9_P5.00mm, J4 Screw_Terminal_9_P5.00mm, J5 Screw_Terminal_9_P5.00mm, K1 G5V-1, K2 G5V-1, Q1 NCE60P04R, Q2 ZXMS6004FFQTA, Q3 ZXMS6004FFQTA, Q4 ZXMS6004FFQTA, Q5 ZXMS6004FFQTA, SW1 TS-1088-AR02016, SW2 TS-1088-AR02016, U1 TD301M485_C5451847, U10 ADS1115IDGS, U11 AT3H4B-CUH-S, U12 AT3H4B-CUH-S, U13 LK1802, U14 AT3H4B-CUH-S, U15 MAX31856MUD+, U16 BL0942, U17 B0303S-1WR3_C7465185, U18 ISO7021DR, U19 ESP32-S3-WROOM-1, U2 AT3H4B-CUH-S, U3 AP63203WU, U5 AT3H4B-CUH-S, U6 AT3H4B-CUH-S, U7 GP8211S-TC50-EW, U8 GP8302-TC50-EW, U9 BTS723GWXUMA1

Commit message: Tarea 5: Enrutado el esp
Parts:
- moved R31 2.14 mm to (139.3, 119.7), turned to 180 degrees
- moved R30 1.88 mm to (139.3, 117.0), turned to 180 degrees
Routing:
- net VDC: track 210.3 -> 263.7 mm
- net /control/OUT_PNP2: track 1.67 -> 49.2 mm, vias 1 -> 2
- net /control/EMRX: track 0.00 -> 44.7 mm, vias 0 -> 3
- net /control/OUT_NPN4: track 3.00 -> 47.6 mm
- net /control/OUT_NPN1: track 14.8 -> 59.0 mm, vias 2 -> 3
- net /control/OUT_NPN3: track 6.68 -> 49.5 mm, vias 2 -> 3
- net /control/OUT_NPN2: track 10.8 -> 52.0 mm, vias 2 -> 3
- net /control/EM_TX: track 0.00 -> 40.5 mm, vias 0 -> 2
- net /control/OUT_PNP1: track 1.55 -> 40.0 mm, vias 1 -> 2
- net /control/OUT-PNP/st2: track 0.00 -> 37.2 mm, vias 0 -> 4
- net /control/OUT-PNP/st1: track 0.00 -> 37.0 mm, vias 0 -> 2
- net /control/RS485-RX: track 0.00 -> 22.3 mm, vias 0 -> 2
- net /control/OUT_RLY1: track 0.00 -> 21.7 mm, vias 0 -> 2
- net /control/OUT_RLY2: track 0.00 -> 21.0 mm
- net /control/RS485-TX: track 0.00 -> 17.2 mm, vias 0 -> 2
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
Commit message: Tarea 5: Enrutado sin corregir errores
Parts:
- moved C33 0.79 mm to (161.6, 86.6)
- moved TP2 0.36 mm to (161.7, 91.4)
- moved TP3 0.36 mm to (146.7, 84.9)
- moved R49 0.21 mm to (161.5, 84.4)
- moved D16 0.18 mm to (161.5, 88.6), turned to 0 degrees
Routing:
- net /control/IN-4-20MA1/OUT: track 0.00 -> 43.5 mm, vias 0 -> 1
- net /control/IN-0-10V1/COM: track 1.52 -> 45.0 mm, vias 1 -> 4
- net /control/IN-0-10V1/OUT3V: track 1.96 -> 44.9 mm
- net /control/IN-0-10V/OUT3V: track 3.01 -> 45.7 mm
- net /control/IN-0-10V/COM: track 3.93 -> 40.2 mm, vias 1 -> 4
- net VDC: track 263.7 -> 299.1 mm, vias 4 -> 6
- net /control/IN-4-20MA/OUT: track 0.00 -> 35.3 mm, vias 0 -> 1
- net GND: track 142.0 -> 173.7 mm, vias 96 -> 113
- net Net-(D10-K): track 0.00 -> 9.74 mm
- net Net-(C33-Pad1): track 0.00 -> 9.48 mm
- net +3.3V: track 50.7 -> 60.0 mm, vias 35 -> 39
- net Net-(D15-K): track 0.00 -> 7.86 mm
- net /control/CON-IN-4-20MA_2: track 0.00 -> 6.25 mm
- net Net-(C12-Pad1): track 0.00 -> 4.69 mm

Commit message: Tarea 5: Finalizada
Parts:
- moved U9 0.41 mm to (103.2, 130.5)
- moved U17 0.24 mm to (185.7, 92.6)
- moved JP1 0.19 mm to (103.3, 88.9)
Routing:
- net /control/OUT_NPN1: track 59.0 -> 44.2 mm, vias 3 -> 2
- net /control/OUT_NPN2: track 52.0 -> 41.3 mm, vias 3 -> 2
- net /control/OUT_NPN3: track 49.5 -> 42.8 mm, vias 3 -> 2
- net VDC: track 299.1 -> 294.6 mm
- net /control/CON-IN_CT_P: track 6.51 -> 9.03 mm
- net /control/CON_OUT_PNP2: track 26.1 -> 27.4 mm
- net /control/CON_OUT_PNP1: track 21.5 -> 22.6 mm
- net /control/TEMP_CS: track 27.8 -> 27.2 mm
- net /control/I2C_SDA: vias 5 -> 4
- net /control/I2C_SCK: vias 5 -> 4
